File: HASSlike Control Pendant.kicad_pcb (KiCad board)
At the start: 2 copper layers, 279 parts, among them SW1 SW_Push, SW10 SW_Push, SW100 SW_Push, SW101 SW_Push, SW102 SW_Push, SW103 SW_Push, SW104 SW_Push, SW105 SW_Push, SW106 SW_Push, SW107 SW_Push, SW108 SW_Push, SW109 SW_Push, SW11 SW_Push, SW110 SW_Push, SW111 SW_Push, SW112 SW_Push, SW113 SW_Push, SW114 SW_Push, SW115 SW_Push, SW116 SW_Push, SW117 SW_Push, SW118 SW_Push, SW119 SW_Push, SW12 SW_Push, SW120 SW_Push, SW121 SW_Push, SW122 SW_Push, SW123 SW_Push, SW124 SW_Push, SW125 SW_Push, SW126 SW_Push, SW127 SW_Push, SW128 SW_Push, SW129 SW_Push, SW13 SW_Push, SW130 SW_Push, SW131 SW_Push, SW132 SW_Push, SW133 SW_Push, SW134 SW_Push, SW135 SW_Push, SW136 SW_Push, SW137 SW_Push, SW138 SW_Push, SW139 SW_Push, SW14 SW_Push, SW15 SW_Push, SW16 SW_Push, SW17 SW_Push, SW18 SW_Push, SW19 SW_Push, SW2 SW_Push, SW20 SW_Push, SW21 SW_Push, SW22 SW_Push, SW23 SW_Push, SW24 SW_Push, SW25 SW_Push, SW26 SW_Push, SW27 SW_Push, SW28 SW_Push, SW29 SW_Push, SW3 SW_Push, SW30 SW_Push, SW31 SW_Push, SW32 SW_Push, SW33 SW_Push, SW34 SW_Push, SW35 SW_Push, SW36 SW_Push, SW37 SW_Push, SW38 SW_Push, SW39 SW_Push, SW4 SW_Push, SW40 SW_Push, SW41 SW_Push, SW42 SW_Push, SW43 SW_Push, SW44 SW_Push, SW45 SW_Push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

Commit message: progress on layout for small-scale proof of concept board
Parts:
- added J1: Conn_01x04_Pin, Connector_JST:JST_SH_BM04B-SRSS-TB_1x04-1MP_P1.00mm_Vertical, B.Cu at (113.2, 177.8)
- added J2: Conn_01x04_Pin, Connector_JST:JST_SH_BM04B-SRSS-TB_1x04-1MP_P1.00mm_Vertical, B.Cu at (106.2, 177.8)
- added U1: MCP23017_SO, Package_SO:SOIC-28W_7.5x17.9mm_P1.27mm, B.Cu at (98.4, 162.5)
- A1: footprint Module:RaspberryPi_Pico_W_SMD_HandSolder -> Module:RaspberryPi_Pico_Common_Unspecified
- D75, D76, D77, D78, D79, D80, D81, D82, D83, D84, D85, D86, D87, D88, D89, D90: moved to B.Cu
- moved D123 457.5 mm to (-97.2, 33.6)
- moved D124 457.5 mm to (-97.2, 38.3)
- moved D125 457.5 mm to (-97.2, 42.9)
- moved D126 457.5 mm to (-97.2, 47.5)
- moved D107 454.2 mm to (-107.0, 33.6)
- moved D108 454.2 mm to (-107.0, 38.3)
- moved D109 454.2 mm to (-107.0, 42.9)
- moved D110 454.2 mm to (-107.0, 47.5)
- moved D111 454.2 mm to (-107.0, 52.1)
- moved D112 454.2 mm to (-107.0, 56.8)
- moved SW123 452.2 mm to (-127.6, 39.0)
- moved SW124 452.2 mm to (-127.6, 54.4)
- moved SW125 452.2 mm to (-127.6, 69.8)
- moved SW126 452.2 mm to (-127.6, 85.2)
- moved D91 451.2 mm to (-116.7, 33.6)
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Connections:
- A1 pad 13: Net-(A1-GND-Pad13) -> GND
- A1 pad 18: Net-(A1-GND-Pad13) -> GND
- A1 pad 23: Net-(A1-GND-Pad13) -> GND
- A1 pad 28: Net-(A1-GND-Pad13) -> GND
- A1 pad 3: Net-(A1-GND-Pad13) -> GND
- A1 pad 36: unconnected-(A1-3V3-Pad36) -> VCC
- A1 pad 38: Net-(A1-GND-Pad13) -> GND
- A1 pad 8: Net-(A1-GND-Pad13) -> GND
- D100 pad 1: ROW7 -> Net-(D100-K)
- D101 pad 1: ROW8 -> Net-(D101-K)
- D102 pad 1: ROW8 -> Net-(D101-K)
- D103 pad 1: ROW8 -> Net-(D101-K)
- D104 pad 1: ROW8 -> Net-(D101-K)
- D105 pad 1: ROW8 -> Net-(D101-K)
- D106 pad 1: ROW8 -> Net-(D101-K)
- D107 pad 1: ROW8 -> Net-(D101-K)
- D108 pad 1: ROW8 -> Net-(D101-K)
- D109 pad 1: ROW8 -> Net-(D101-K)
- D110 pad 1: ROW8 -> Net-(D101-K)
- D111 pad 1: ROW9 -> Net-(D111-K)
- D112 pad 1: ROW9 -> Net-(D111-K)
- D113 pad 1: ROW9 -> Net-(D111-K)
- D114 pad 1: ROW9 -> Net-(D111-K)
- D115 pad 1: ROW9 -> Net-(D111-K)
- D116 pad 1: ROW9 -> Net-(D111-K)
- D117 pad 1: ROW9 -> Net-(D111-K)
- D118 pad 1: ROW9 -> Net-(D111-K)
- D119 pad 1: ROW9 -> Net-(D111-K)
- D120 pad 1: ROW9 -> Net-(D111-K)
- D121 pad 1: ROW10 -> Net-(D121-K)
- D122 pad 1: ROW10 -> Net-(D121-K)
- D123 pad 1: ROW10 -> Net-(D121-K)
- D124 pad 1: ROW10 -> Net-(D121-K)
- D125 pad 1: ROW10 -> Net-(D121-K)
- D126 pad 1: ROW10 -> Net-(D121-K)
- D127 pad 1: ROW10 -> Net-(D121-K)
- D128 pad 1: ROW10 -> Net-(D121-K)
- D129 pad 1: ROW10 -> Net-(D121-K)
- D130 pad 1: ROW10 -> Net-(D121-K)
- D75 pad 1: ROW7 -> /4x4Test/Row1
- D76 pad 1: ROW7 -> /4x4Test/Row1
- D77 pad 1: ROW7 -> /4x4Test/Row1
- D78 pad 1: ROW7 -> /4x4Test/Row1
- D79 pad 1: ROW8 -> /4x4Test/Row2
- D80 pad 1: ROW8 -> /4x4Test/Row2
- D81 pad 1: ROW8 -> /4x4Test/Row2
- D82 pad 1: ROW8 -> /4x4Test/Row2
- D83 pad 1: ROW9 -> /4x4Test/Row3
- D84 pad 1: ROW9 -> /4x4Test/Row3
- D85 pad 1: ROW9 -> /4x4Test/Row3
- D86 pad 1: ROW9 -> /4x4Test/Row3
- D87 pad 1: ROW10 -> /4x4Test/Row4
- D88 pad 1: ROW10 -> /4x4Test/Row4
- D89 pad 1: ROW10 -> /4x4Test/Row4
- D90 pad 1: ROW10 -> /4x4Test/Row4
- D91 pad 1: ROW7 -> Net-(D100-K)
- D92 pad 1: ROW7 -> Net-(D100-K)
- D93 pad 1: ROW7 -> Net-(D100-K)
- D94 pad 1: ROW7 -> Net-(D100-K)
- D95 pad 1: ROW7 -> Net-(D100-K)
- D96 pad 1: ROW7 -> Net-(D100-K)
- D97 pad 1: ROW7 -> Net-(D100-K)
- D98 pad 1: ROW7 -> Net-(D100-K)
- D99 pad 1: ROW7 -> Net-(D100-K)
- SW100 pad 1: COL14 -> Net-(SW100-Pad1)
- SW101 pad 1: COL5 -> unconnected-(SW101-Pad1)
- SW102 pad 1: COL6 -> Net-(SW102-Pad1)
- SW103 pad 1: COL7 -> Net-(SW103-Pad1)
- SW104 pad 1: COL8 -> Net-(SW104-Pad1)
- SW105 pad 1: COL9 -> Net-(SW105-Pad1)
- SW106 pad 1: COL10 -> Net-(SW106-Pad1)
- SW107 pad 1: COL11 -> Net-(SW107-Pad1)
- SW108 pad 1: COL12 -> Net-(SW108-Pad1)
- SW109 pad 1: COL13 -> Net-(SW109-Pad1)
- SW110 pad 1: COL14 -> Net-(SW100-Pad1)
- SW111 pad 1: COL5 -> unconnected-(SW111-Pad1)
- SW112 pad 1: COL6 -> Net-(SW102-Pad1)
- SW113 pad 1: COL7 -> Net-(SW103-Pad1)
- SW114 pad 1: COL8 -> Net-(SW104-Pad1)
- SW115 pad 1: COL9 -> Net-(SW105-Pad1)
- SW116 pad 1: COL10 -> Net-(SW106-Pad1)
- SW117 pad 1: COL11 -> Net-(SW107-Pad1)
- SW118 pad 1: COL12 -> Net-(SW108-Pad1)
- SW119 pad 1: COL13 -> Net-(SW109-Pad1)
- SW120 pad 1: COL14 -> Net-(SW100-Pad1)
- SW121 pad 1: COL5 -> unconnected-(SW121-Pad1)
- SW122 pad 1: COL6 -> Net-(SW102-Pad1)
- SW123 pad 1: COL7 -> Net-(SW103-Pad1)
- SW124 pad 1: COL8 -> Net-(SW104-Pad1)
- SW125 pad 1: COL9 -> Net-(SW105-Pad1)
- SW126 pad 1: COL10 -> Net-(SW106-Pad1)
- SW127 pad 1: COL11 -> Net-(SW107-Pad1)
- SW128 pad 1: COL12 -> Net-(SW108-Pad1)
- SW129 pad 1: COL13 -> Net-(SW109-Pad1)
- SW130 pad 1: COL14 -> Net-(SW100-Pad1)
- SW75 pad 1: COL1 -> /4x4Test/Col1
- SW76 pad 1: COL2 -> /4x4Test/Col2
- SW77 pad 1: COL3 -> /4x4Test/Col3
- SW78 pad 1: COL4 -> /4x4Test/Col4
- SW79 pad 1: COL1 -> /4x4Test/Col1
- SW80 pad 1: COL2 -> /4x4Test/Col2
- SW81 pad 1: COL3 -> /4x4Test/Col3
- SW82 pad 1: COL4 -> /4x4Test/Col4
- SW83 pad 1: COL1 -> /4x4Test/Col1
- SW84 pad 1: COL2 -> /4x4Test/Col2
- SW85 pad 1: COL3 -> /4x4Test/Col3
- SW86 pad 1: COL4 -> /4x4Test/Col4
- SW87 pad 1: COL1 -> /4x4Test/Col1
- SW88 pad 1: COL2 -> /4x4Test/Col2
- SW89 pad 1: COL3 -> /4x4Test/Col3
- SW90 pad 1: COL4 -> /4x4Test/Col4
- SW91 pad 1: COL5 -> unconnected-(SW91-Pad1)
- SW92 pad 1: COL6 -> Net-(SW102-Pad1)
- SW93 pad 1: COL7 -> Net-(SW103-Pad1)
- SW94 pad 1: COL8 -> Net-(SW104-Pad1)
- SW95 pad 1: COL9 -> Net-(SW105-Pad1)
- SW96 pad 1: COL10 -> Net-(SW106-Pad1)
- SW97 pad 1: COL11 -> Net-(SW107-Pad1)
- SW98 pad 1: COL12 -> Net-(SW108-Pad1)
- SW99 pad 1: COL13 -> Net-(SW109-Pad1)
Routing:
- net /4x4Test/Col1: track 0.00 -> 163.8 mm, vias 0 -> 1
- net /4x4Test/Col2: track 0.00 -> 142.9 mm, vias 0 -> 1
- net /4x4Test/Col3: track 0.00 -> 124.9 mm, vias 0 -> 1
- net /4x4Test/Row4: track 0.00 -> 107.3 mm
- net /4x4Test/Row1: track 0.00 -> 95.3 mm
- net /4x4Test/Row3: track 0.00 -> 91.7 mm
- net /4x4Test/Col4: track 0.00 -> 82.3 mm, vias 0 -> 1
- net /4x4Test/Row2: track 0.00 -> 79.1 mm
- net GND: track 0.00 -> 50.8 mm
- net VCC: track 0.00 -> 36.9 mm
- net /SCL: track 0.00 -> 22.3 mm
- net /SDA: track 0.00 -> 19.9 mm
- net Net-(D78-A): track 0.00 -> 9.60 mm
- net Net-(D82-A): track 0.00 -> 9.60 mm
- net Net-(D77-A): track 0.00 -> 9.60 mm
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Other:
- board text added: "TODO: Populate LEDS Select and add encoder"
- board text added: "TODO: mouse bites cut here"
